File: pcb/D1_mini_shield_client/D1_mini_shield_client.kicad_pcb (KiCad board)
At the start: 2 copper layers, 7 parts, among them J1 BME280, J2 Battery, U1 WeMos_mini

Commit message: Update pcb.
Parts:
- R2: value 4k7 -> 470
Other:
- net class Default removed
